Commit message: update code

File: humanoidGym/resources/robots/miniloong_v4_12dof/urdf/miniloong_v4_12dof_c_new_V41.urdf (robot description, URDF)
Before this commit: robot miniloong_v3, 23 links, 22 joints
Links:
- link link_left_ankle_roll: geometry collision sphere radius=0.005; collision sphere radius=0.005
- link link_right_ankle_roll: geometry collision sphere radius=0.005; collision sphere radius=0.005

File: humanoidGym/resources/robots/miniloong_v4_12dof/urdf/miniloong_v4_12dof_c_new_V41_1.urdf (robot description, URDF)
Before this commit: robot miniloong_v3, 23 links, 22 joints
Links:
- link link_left_ankle_roll: geometry collision sphere radius=0.005; collision sphere radius=0.005
- link link_right_ankle_roll: geometry collision sphere radius=0.005; collision sphere radius=0.005
